File: MCU/MCU.kicad_pcb (KiCad board)
At the start: 2 copper layers, 100 x 97.8 mm, 173 parts, among them J101 Power_Conn, J102 MCU_UART_Conn, J103 MCU_CAM_UART_Conn, J104 920MHz_Conn, J105 I2C_Conn, J106 I2C_Conn, J107 Motor_Conn, J108 CdS_Conn, J109 Power_EN_Conn, J110 I2C_Conn, J111 UART_Conn, J112 GPS_UART_Conn, J113 M_PWM, J114 I2C_Conn, J115 I2C_Conn, J116 I2C_Conn, J117 CAM_Conn, J118 Power_Conn, J119 Power_Conn, J120 Power_Conn, J121 MCU_Power, J122 MCU_Power, J123 Power_EN, J124 Motor_Power, J125 MCU_Power, J126 Micro_SD_Card_Det_Hirose_DM3AT, J127 MCU_Power, J128 MCU_Power, J201 FlightPin, J202 Heater, J301 Battery, J302 Battery, J401 M_Power_Conn, J402 M1, J403 M2, J801 Conn_Coaxial, Q301 2SB1198K, Q302 2SB1198K, Q303 2N7002, Q304 2SB1198K, Q305 2N7002, Q306 2SC2412K, Q307 PJA3404A, Q308 PJA3404A, U101 ESP32-S3-WROOM-1U-N4R8, U102 ESP32-S3-WROOM-1U-N4R8, U201 TPS564252, U202 TPS564252, U203 TPS22810DBV, U301 S-8209ABB-T8T1U, U302 S-8209ABB-T8T1U, U401 DRV8835, U601 AE-BME280, U701 BNO055 FusionModule, U801 NEO-M9N

Commit message: Update: 隙間を詰めてみた
でも大きいなあ
裏面が結構空いてる
Parts:
- removed G*** (x2): LOGO, LOGO
- removed J101, J118, J119, J120: Power_Conn, Connector_JST:JST_XH_B2B-XH-A_1x02_P2.50mm_Vertical
- removed J107: Motor_Conn, Connector_JST:JST_XH_B8B-XH-A_1x08_P2.50mm_Vertical
- removed J108: CdS_Conn, Connector_JST:JST_XH_B3B-XH-A_1x03_P2.50mm_Vertical
- removed J109: Power_EN_Conn, Connector_JST:JST_XH_B3B-XH-A_1x03_P2.50mm_Vertical
- removed J110, J114, J115, J116: I2C_Conn, Connector_JST:JST_XH_B3B-XH-A_1x03_P2.50mm_Vertical
- removed J111: UART_Conn, Connector_JST:JST_XH_B3B-XH-A_1x03_P2.50mm_Vertical
- removed J112: GPS_UART_Conn, Connector_JST:JST_XH_B3B-XH-A_1x03_P2.50mm_Vertical
- removed J113: M_PWM, Connector_JST:JST_XH_B8B-XH-A_1x08_P2.50mm_Vertical
- removed J123: Power_EN, Connector_JST:JST_XH_B3B-XH-A_1x03_P2.50mm_Vertical
- removed J125, J127, J128: MCU_Power, Connector_JST:JST_XH_B2B-XH-A_1x02_P2.50mm_Vertical
- removed REF** (x13): Mousebite_5x2mm, Project:Mousebite_5x2mm
- removed REF** (x19): Mousebite_5x1.6mm, Project:Mousebite_5x1.6mm
- removed REF** (x2): MountingHole_3.2mm_M3, MountingHole:MountingHole_3.2mm_M3
- moved U401 16.5 mm to (161.7, 125.4)
- moved J402 16.5 mm to (169.4, 134.4)
- moved J403 16.5 mm to (154.4, 134.4)
- moved C401 16.5 mm to (158.9, 124.4)
- moved C402 16.5 mm to (158.9, 126.4)
- moved J401 16.5 mm to (154.4, 127.4)
- moved BT801 12.9 mm to (126.9, 120.5)
- moved C801 12.9 mm to (125.9, 123.0)
- moved C803 12.9 mm to (127.9, 123.0)
- moved D801 12.9 mm to (126.9, 118.0)
- moved JP801 12.9 mm to (112.9, 127.0)
- moved R802 12.9 mm to (112.9, 124.5)
- moved R803 12.9 mm to (126.9, 123.0)
- moved U801 12.9 mm to (121.4, 132.5)
- moved C802 12.9 mm to (110.2, 134.9)
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Connections:
- BT801 pad 2: /GPS/GND -> GND
- C101 pad 2: /GND -> GND
- C102 pad 2: /GND -> GND
- C103 pad 2: /GND -> GND
- C104 pad 2: /GND -> GND
- C105 pad 2: /GND -> GND
- C201 pad 2: /Power/GND -> GND
- C202 pad 2: /Power/GND -> GND
- C203 pad 1: /Power/3V3 -> /VCC
- C204 pad 1: /Power/3V3 -> /VCC
- C204 pad 2: /Power/GND -> GND
- C205 pad 1: /Power/3V3 -> /VCC
- C205 pad 2: /Power/GND -> GND
- C206 pad 1: /Power/3V3 -> /VCC
- C206 pad 2: /Power/GND -> GND
- C207 pad 2: /Power/GND -> GND
- C208 pad 2: /Power/GND -> GND
- C210 pad 2: /Power/GND -> GND
- C211 pad 2: /Power/GND -> GND
- C212 pad 2: /Power/GND -> GND
- C213 pad 2: /Power/GND -> GND
- C214 pad 2: /Power/GND -> GND
- C215 pad 2: /Power/GND -> GND
- C401 pad 1: /MD/VCC -> /VCC
- C401 pad 2: /MD/GND -> GND
- C402 pad 2: /MD/GND -> GND
- C801 pad 1: /GPS/VCC -> /VCC
- C801 pad 2: /GPS/GND -> GND
- C802 pad 2: /GPS/GND -> GND
- C803 pad 2: /GPS/GND -> GND
- D801 pad 2: /GPS/VCC -> /VCC
- J102 pad 5: /GND -> GND
- J103 pad 5: /GND -> GND
- J104 pad 3: /GND -> GND
- J105 pad 3: /GND -> GND
- J106 pad 3: /GND -> GND
- J117 pad 2: /GND -> GND
- J121 pad 1: /Power/3V3 -> /VCC
- J121 pad 2: /Power/GND -> GND
- J122 pad 1: /Power/3V3 -> /VCC
- J122 pad 2: /Power/GND -> GND
- J124 pad 2: /Power/GND -> GND
- J126 pad 6: /GND -> GND
- J201 pad 1: /Power/FP -> /FP
- J201 pad 2: /Power/GND -> GND
- J202 pad 2: /Power/GND -> GND
- J401 pad 2: /MD/GND -> GND
- J801 pad 2: /GPS/GND -> GND
- JP601 pad 3: /I2C Sensors/VCC -> /VCC
- JP801 pad 1: /GPS/GND -> GND
- L201 pad 2: /Power/3V3 -> /VCC
- Q307 pad 2: /Power/GND -> GND
- R201 pad 1: /Power/3V3 -> /VCC
- R203 pad 1: /Power/3V3 -> /VCC
- R205 pad 2: /Power/GND -> GND
- R206 pad 2: /Power/GND -> GND
- R210 pad 2: /Power/GND -> GND
- R211 pad 1: /Power/3V3 -> /VCC
- R211 pad 2: /Power/FP -> /FP
- R212 pad 1: /Power/PC_Sep -> /PC_Sep
- R212 pad 2: /Power/GND -> GND
- R313 pad 1: /Power/GND -> GND
- R315 pad 2: /Power/GND -> GND
- R802 pad 1: /GPS/VCC -> /VCC
- U101 pad 1: /GND -> GND
- U101 pad 12: /CdS -> unconnected-(U101-GPIO8/TOUCH8/ADC1_CH7/SUBSPICS1-Pad12)
- U101 pad 40: /GND -> GND
- U101 pad 41: /GND -> GND
- U102 pad 1: /GND -> GND
- U102 pad 40: /GND -> GND
- U102 pad 41: /GND -> GND
- U201 pad 3: /Power/GND -> GND
- U202 pad 3: /Power/GND -> GND
- U202 pad 5: /Power/Motor_P_EN -> /Motor_P_EN
- U203 pad 2: /Power/GND -> GND
- U203 pad 3: /Power/PC_Sep -> /PC_Sep
- U401 pad 10: /MD/AIN1 -> /MA1
- U401 pad 11: /MD/GND -> GND
- U401 pad 12: /MD/VCC -> /VCC
- U401 pad 13: /MD/GND -> GND
- U401 pad 6: /MD/GND -> GND
- U401 pad 7: /MD/BIN2 -> /MB2
- U401 pad 8: /MD/BIN1 -> /MB1
- U401 pad 9: /MD/AIN2 -> /MA2
- U601 pad 1: /I2C Sensors/VCC -> /VCC
- U601 pad 3: /I2C Sensors/VCC -> /VCC
- U601 pad 4: /I2C Sensors/SDA -> /I2C1SDA
- U601 pad 6: /I2C Sensors/SCK -> /I2C1SCL
- U701 pad 1: /I2C Sensors/VCC -> /VCC
- U701 pad 3: /I2C Sensors/SDA -> /I2C1SDA
- U701 pad 4: /I2C Sensors/SCK -> /I2C1SCL
- U801 pad 10: /GPS/GND -> GND
- U801 pad 12: /GPS/GND -> GND
- U801 pad 13: /GPS/GND -> GND
- U801 pad 18: /GPS/SDA -> /I2C1SDA
- U801 pad 19: /GPS/SCL -> /I2C1SCL
- U801 pad 20: /GPS/GPS_TX -> /U1RXD
- U801 pad 21: /GPS/GPS_RX -> /U1TXD
- U801 pad 23: /GPS/VCC -> /VCC
- U801 pad 24: /GPS/GND -> GND
- U801 pad 7: /GPS/GND -> GND
Routing:
- net GND: track 49.4 -> 515.5 mm, vias 26 -> 54
- net /GND: track 312.2 -> 0.00 mm, vias 88 -> 0
- net /Power/GND: track 169.0 -> 0.00 mm, vias 37 -> 0
- net /VCC: track 199.0 -> 328.6 mm, vias 12 -> 17
- net /GPS/GND: track 113.6 -> 0.00 mm, vias 51 -> 0
- net /Power/3V3: track 79.3 -> 0.00 mm, vias 3 -> 0
- net /CdS: track 46.7 -> 0.00 mm, vias 2 -> 0
- net /MD/GND: track 39.8 -> 0.00 mm, vias 32 -> 0
- net /I2C Sensors/SCK: track 37.9 -> 0.00 mm, vias 1 -> 0
- net /I2C Sensors/VCC: track 37.6 -> 0.00 mm
- net /I2C Sensors/SDA: track 35.3 -> 0.00 mm, vias 1 -> 0
- net /GPS/VCC: track 31.2 -> 0.00 mm, vias 2 -> 0
- net /GPS/SDA: track 30.7 -> 0.00 mm, vias 1 -> 0
- net /GPS/SCL: track 30.1 -> 0.00 mm, vias 1 -> 0
- net /Power/PC_Sep: track 25.5 -> 0.00 mm, vias 1 -> 0
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- removed copper zone on B.Cu, net /GND
- removed copper zone on F.Cu, net /GND
- removed copper zone on B.Cu, net /GPS/GND
- removed copper zone on F.Cu, net /GPS/GND
- removed copper zone on B.Cu, net /MD/GND
- removed copper zone on F.Cu, net /MD/GND
- removed copper zone on F.Cu, net /Power/3V
- removed copper zone on F.Cu, net /Power/3V3
- removed copper zone on B.Cu, net /Power/GND
- removed copper zone on F.Cu, net /Power/GND
- removed copper zone on F.Cu, net Net-(J301-Pin_2)
- removed copper zone on F.Cu, net Net-(U201-SW)
- removed copper zone on F.Cu, net Net-(U202-SW)
Other:
- board outline removed
- board text removed: "Denshiruko"
- board text removed: "Designed by"
- board text removed: "Ver1.0"
- board text removed: "ぶっとび組"
