File: cansat2026/BMS.kicad_sch (KiCad schematic)
At the start: 35 parts, among them J301 Battery, J302 Battery, Q301 2SB1198K, Q302 2SB1198K, Q303 2N7002, Q304 2SB1198K, Q305 2N7002, Q306 2SC2412K, Q307 PJA3404A, Q308 PJA3404A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

Commit message: Update: いろいろした
無線変えた
カメラのコネクタ変えた
i2cセンサ変えた
電源変えた:1.2V,3.8V,3.3V
IOエキスパンダ追加
FPGA追加
Parts:
- C301, C303: footprint Capacitor_SMD:C_0603_1608Metric -> Capacitor_SMD:C_0402_1005Metric; LCSC Part C14663 -> C307331

Commit message: Update: MDと電源とか
MD変えた
モーター電源と主電源
Parts:
- C301, C303: LCSC Part C307331 -> C1525
Changed lines of the file:
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@@
 			)
 		)
-		(property "LCSC Part" "C307331"
+		(property "LCSC Part" "C1525"
 			(at 213.36 115.57 0)
 			(hide yes)
@@
 			)
 		)
-		(property "LCSC Part" "C307331"
+		(property "LCSC Part" "C1525"
 			(at 213.36 77.47 0)
 			(hide yes)

Commit message: Update: 完成した
Parts:
- J301, J302: footprint Connector_JST:JST_XH_B2B-XH-A_1x02_P2.50mm_Vertical -> Connector_JST:JST_VH_B2P-VH_1x02_P3.96mm_Vertical; 秋月 Part (none) -> 112815
- Q301, Q302, Q304: Mouser Part 755-2SB1198KT146R -> (none)
- Q306: DigiKey Part (none) -> 2SC2412KT146R; Mouser Part 755-2SC2412KT146R -> (none)
- Q307, Q308: DigiKey Part (none) -> PJA3404A_R1_00001
- R306, R312: DigiKey Part (none) -> RCS120651R0JNEA
Changed lines of the file:
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@@
 			)
 		)
-		(property "DigiKey Part" ""
+		(property "DigiKey Part" "RCS120651R0JNEA"
 			(at 224.79 83.82 90)
 			(hide yes)
@@
 			)
 		)
-		(property "Mouser Part" "755-2SB1198KT146R"
+		(property "Mouser Part" ""
 			(at 86.36 71.12 0)
 			(hide yes)
@@
 			)
 		)
-		(property "DigiKey Part" ""
+		(property "DigiKey Part" "PJA3404A_R1_00001"
 			(at 106.68 140.97 90)
 			(hide yes)
@@
 			)
 		)
-		(property "Footprint" "Connector_JST:JST_XH_B2B-XH-A_1x02_P2.50mm_Vertical"
+		(property "Footprint" "Connector_JST:JST_VH_B2P-VH_1x02_P3.96mm_Vertical"
 			(at 246.38 129.54 0)
 			(hide yes)
@@
 			)
 		)
+		(property "秋月 Part" "112815"
+			(at 246.38 129.54 0)
+			(hide yes)
+			(show_name no)
+			(do_not_autoplace no)
+			(effects
+				(font
+					(size 1.27 1.27)
+				)
+			)
+		)
 		(pin "1"
 		)
@@
 			)
 		)
-		(property "Mouser Part" "755-2SB1198KT146R"
+		(property "Mouser Part" ""
 			(at 127 118.11 0)
 			(hide yes)
@@
 			)
 		)
-		(property "DigiKey Part" ""
+		(property "DigiKey Part" "RCS120651R0JNEA"
 			(at 224.79 121.92 90)
 			(hide yes)
@@
 			)
 		)
-		(property "Mouser Part" "755-2SB1198KT146R"
+		(property "Mouser Part" ""
 			(at 114.3 71.12 0)
 			(hide yes)
@@
 			)
 		)
-		(property "Footprint" "Connector_JST:JST_XH_B2B-XH-A_1x02_P2.50mm_Vertical"
+		(property "Footprint" "Connector_JST:JST_VH_B2P-VH_1x02_P3.96mm_Vertical"
 			(at 246.38 91.44 0)
 			(hide yes)
@@
 			)
 		)
+		(property "秋月 Part" "112815"
+			(at 246.38 91.44 0)
+			(hide yes)
+			(show_name no)
+			(do_not_autoplace no)
+			(effects
+				(font
+					(size 1.27 1.27)
+				)
+			)
+		)
 		(pin "1"
 		)
@@
 			)
 		)
-		(property "DigiKey Part" ""
+		(property "DigiKey Part" "PJA3404A_R1_00001"
 			(at 78.74 140.97 90)
 			(hide yes)
@@
 			)
 		)
-		(property "Mouser Part" "755-2SC2412KT146R"
+		(property "Mouser Part" ""
 			(at 139.7 138.43 0)
 			(hide yes)
@@
 			)
 		)
-		(property "DigiKey Part" ""
+		(property "DigiKey Part" "2SC2412KT146R"
 			(at 139.7 138.43 0)
 			(hide yes)
