File: cansat2026/BMS.kicad_sch (KiCad schematic)
At the start: 35 parts, among them J301 Battery, J302 Battery, Q301 2SB1198K, Q302 2SB1198K, Q303 2N7002, Q304 2SB1198K, Q305 2N7002, Q306 2SC2412K, Q307 PJA3404A, Q308 PJA3404A, U301 S-8209ABB-T8T1U, U302 S-8209ABB-T8T1U

Commit message: ARLISSに作り直した
Parts:
- R307, R314: footprint Resistor_SMD:R_0402_1005Metric -> Resistor_SMD:R_0603_1608Metric; LCSC Part C26082 -> C7250
Changed lines of the file:
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@@
 			)
 		)
-		(property "Footprint" "Resistor_SMD:R_0402_1005Metric"
+		(property "Footprint" "Resistor_SMD:R_0603_1608Metric"
 			(at 193.04 91.44 0)
 			(hide yes)
@@
 			)
 		)
-		(property "LCSC Part" "C26082"
+		(property "LCSC Part" "C7250"
 			(at 193.04 91.44 0)
 			(hide yes)
@@
 			)
 		)
-		(property "Footprint" "Resistor_SMD:R_0402_1005Metric"
+		(property "Footprint" "Resistor_SMD:R_0603_1608Metric"
 			(at 193.04 129.54 0)
 			(hide yes)
@@
 			)
 		)
-		(property "LCSC Part" "C26082"
-			(at 193.04 129.54 0)
-			(hide yes)
+		(property "LCSC Part" "C7250"
+			(at 193.04 129.54 0)
+			(hide yes)
