File: cansat2026/IMU.kicad_sch (KiCad schematic)
At the start: 1 part, among them U701 BNO055 FusionModule

Commit message: Update: いろいろした
無線変えた
カメラのコネクタ変えた
i2cセンサ変えた
電源変えた:1.2V,3.8V,3.3V
IOエキスパンダ追加
FPGA追加
Parts:
- removed U701: BNO055 FusionModule, Project:BNO055-FusionModule, symbol Project:BNO055-FusionModule
- added JP701: I2C Addr, Jumper:SolderJumper-3_P1.3mm_Bridged12_RoundedPad1.0x1.5mm_NumberLabels, symbol Jumper:SolderJumper_3_Bridged12
- added U701: AE-LSM6DSV16X, Project:AE-LSM6DSV16X, symbol Project:AE-LSM6DSV16X
Connections:
- net GND: now also JP701.3 (B), U701.1 (SDX), U701.2 (SCX), U701.5 (GND)
- net SCK: now also U701.10 (SCL)
- net SDA: now also U701.11 (SDA)
- net VCC: now also JP701.1 (A), U701.6 (VDD)
- new net: JP701.2 (C), U701.12 (SDO/SA0)
- no-connect marks 3 -> 5

Commit message: Update: 完成した
Parts:
- removed U701: AE-LSM6DSV16X, Project:AE-LSM6DSV16X, symbol Project:AE-LSM6DSV16X
- added C701, C702: 100nF, Capacitor_SMD:C_0402_1005Metric, symbol Device:C
- added U701: LSM6DSV, Package_LGA:LGA-14_3x2.5mm_P0.5mm_LayoutBorder3x4y, symbol Sensor_Motion:LSM6DS3
Connections:
- net GND: now also C701.2, C702.2, U701.2 (SDX), U701.3 (SCX), U701.6 (GND), U701.7 (GND)
- net SCK: now also U701.13 (SCL)
- net SDA: now also U701.14 (SDA)
- net VCC: now also C701.1, C702.1, U701.12 (CS), U701.5 (VDDIO), U701.8 (VDD)
- net at JP701.2 (C): now also U701.1 (SDO/SA0)
- no-connect marks 5 -> 2
