File: cansat2026/IMU.kicad_sch (KiCad schematic)
At the start: 4 parts, among them U701 LSM6DSV

Commit message: ARLISSに作り直した
Parts:
- U701: LCSC Part C5267399 -> (none)
Changed lines of the file:
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@@
 			)
 		)
-		(property "LCSC Part" "C5267399"
+		(property "LCSC Part" ""
 			(at 165.1 101.6 0)
 			(hide yes)
