File: cansat2026/MCU.kicad_sch (KiCad schematic)
At the start: 17 parts, among them U101 ESP32-S3-WROOM-1U-N4R8, U102 ESP32-S3-WROOM-1U-N4R8

Commit message: Update: いろいろした
無線変えた
カメラのコネクタ変えた
i2cセンサ変えた
電源変えた:1.2V,3.8V,3.3V
IOエキスパンダ追加
FPGA追加
Parts:
- added C906: 1uF, Capacitor_SMD:C_0402_1005Metric, symbol Device:C_Small
- added R901: 10k, Resistor_SMD:R_0402_1005Metric, symbol Device:R_Small
- added R909: 4.7k, Resistor_SMD:R_0402_1005Metric, symbol Device:R
- added R913: 10k, Resistor_SMD:R_0402_1005Metric, symbol Device:R
- added U903: AW9523B, Package_DFN_QFN:QFN-24-1EP_4x4mm_P0.5mm_EP2.7x2.7mm, symbol Interface_Expansion:AW9523B
- renumbered C101 to C901, C102 to C902, C103 to C903, C104 to C904, C105 to C905, R101 to R902, R102 to R903, R103 to R904, R104 to R905, R105 to R906, R106 to R907, R107 to R908, R109 to R910, R110 to R911, R111 to R912, U101 to U901, U102 to U902
Connections:
- net CAM_PIN_D0: now also U902.4 (GPIO4/TOUCH4/ADC1_CH3); no longer U902.19 (GPIO11/TOUCH11/ADC2_CH0/FSPID/FSPIIO5/SUBSPID)
- net CAM_PIN_D1: now also U902.5 (GPIO5/TOUCH5/ADC1_CH4); no longer U902.17 (GPIO9/TOUCH9/ADC1_CH8/FSPIHD/SUBSPIHD)
- net CAM_PIN_D2: now also U902.6 (GPIO6/TOUCH6/ADC1_CH5); no longer U902.12 (GPIO8/TOUCH8/ADC1_CH7/SUBSPICS1)
- net CAM_PIN_D3: now also U902.7 (GPIO7/TOUCH7/ADC1_CH6); no longer U902.18 (GPIO10/TOUCH10/ADC1_CH9/FSPICS0/FSPIIO4/SUBSPICS0)
- net CAM_PIN_D4: now also U902.8 (GPIO15/U0RTS/ADC2_CH4/XTAL_32K_P); no longer U902.20 (GPIO12/TOUCH12/ADC2_CH1/FSPICLK/FSPIIO6/SUBSPICLK)
- net CAM_PIN_D5: now also U902.9 (GPIO16/U0CTS/ADC2_CH5/XTAL_32K_N); no longer U902.11 (GPIO18/U1RXD/ADC2_CH7/CLK_OUT3)
- net CAM_PIN_D7: now also U902.11 (GPIO18/U1RXD/ADC2_CH7/CLK_OUT3); no longer U902.9 (GPIO16/U0CTS/ADC2_CH5/XTAL_32K_N)
- net CAM_PIN_HREF: now also U902.17 (GPIO9/TOUCH9/ADC1_CH8/FSPIHD/SUBSPIHD); no longer U902.7 (GPIO7/TOUCH7/ADC1_CH6)
- net CAM_PIN_PCLK: now also U902.12 (GPIO8/TOUCH8/ADC1_CH7/SUBSPICS1); no longer U902.21 (GPIO13/TOUCH13/ADC2_CH2/FSPIQ/FSPIIO7/SUBSPIQ)
- net CAM_PIN_PWDN: now also U902.23 (GPIO21); no longer U902.31 (GPIO38/FSPIWP/SUBSPIWP)
- net CAM_PIN_RESET: now also U902.31 (GPIO38/FSPIWP/SUBSPIWP); no longer U902.23 (GPIO21)
- net CAM_PIN_SIOC: now also U902.25 (GPIO48/SPICLK_N/SUBSPICLK_N_DIFF); no longer U902.5 (GPIO5/TOUCH5/ADC1_CH4)
- net CAM_PIN_SIOD: now also U902.24 (GPIO47/SPICLK_P/SUBSPICLK_P_DIFF); no longer U902.4 (GPIO4/TOUCH4/ADC1_CH3)
- net CAM_PIN_VSYNC: now also U902.22 (GPIO14/TOUCH14/ADC2_CH3/FSPIWP/FSPIDQS/SUBSPIWP); no longer U902.6 (GPIO6/TOUCH6/ADC1_CH5)
- net CAM_PIN_XCLK: no longer U902.8 (GPIO15/U0RTS/ADC2_CH4/XTAL_32K_P)
- net FP: now also U903.5 (P0_0); no longer U901.31 (GPIO38/FSPIWP/SUBSPIWP)
- net GND: now also C906.2, R901.2, R913.2, U903.24 (AD1), U903.25 (GND), U903.9 (GND)
- net I2C1SCL: now also U903.19 (SCL)
- net I2C1SDA: now also U903.20 (SDA)
- net MCU_CAM_EN: now also R901.1, U903.14 (P1_4); no longer U901.24 (GPIO47/SPICLK_P/SUBSPICLK_P_DIFF)
- net Motor_P_EN: now also U903.16 (P1_6); no longer U901.25 (GPIO48/SPICLK_N/SUBSPICLK_N_DIFF)
- net PC_Sep: now also U903.10 (P0_4); no longer U901.23 (GPIO21)
- net VCC: now also C906.1, R909.1, U903.18 (AD0), U903.21 (VCC)
- net FPGA_~{CRESET}: now reaches U902.34 (MTDI/GPIO41/CLK_OUT1)
- net FPGA_CDONE: now reaches U902.35 (MTMS/GPIO42)
- new net COM_AUX: U901.23 (GPIO21)
- new net COM_M0: U903.11 (P0_5)
- new net COM_M1: U903.12 (P0_6)
- new net COM_P_EN: U903.15 (P1_5)
- new net FPGA_SPI_MISO: U902.20 (GPIO12/TOUCH12/ADC2_CH1/FSPICLK/FSPIIO6/SUBSPICLK)
- new net FPGA_SPI_MOSI: U902.19 (GPIO11/TOUCH11/ADC2_CH0/FSPID/FSPIIO5/SUBSPID)
- new net FPGA_SPI_SCK: U902.18 (GPIO10/TOUCH10/ADC1_CH9/FSPICS0/FSPIIO4/SUBSPICS0)
- new net FPGA_SPI_SS: R913.1, U902.21 (GPIO13/TOUCH13/ADC2_CH2/FSPIQ/FSPIIO7/SUBSPIQ)
- new net IOEX_~{INT}: R909.2, U901.24 (GPIO47/SPICLK_P/SUBSPICLK_P_DIFF), U903.22 (~{INT})
- new net IOEX_~{RST}: U901.25 (GPIO48/SPICLK_N/SUBSPICLK_N_DIFF), U903.23 (~{RST})
- no-connect marks 28 -> 33
Other:
- added sheet FPGA (FPGA.kicad_sch)
- note added: "H"
- note added: "Hi-Z"
- note added: "L"

Commit message: Update: MDと電源とか
MD変えた
モーター電源と主電源
Parts:
- added D901, D902, D903: LED, LED_SMD:LED_0603_1608Metric, symbol Device:LED_Small
- added R903: 100k, Resistor_SMD:R_0402_1005Metric, symbol Device:R
- added R914, R915, R916: 1k, Resistor_SMD:R_0402_1005Metric, symbol Device:R_Small
- added SW901: SW_SPST, Project:IS-1235-G, symbol Switch:SW_SPST
- renumbered R903 to R904, R904 to R905, R905 to R906, R906 to R907, R907 to R908, R908 to R909, R909 to R910, R910 to R911, R911 to R912, R912 to R913, R913 to R917
Connections:
- net PC_Sep is gone; now on net MCU_CAM_EN: U903.10 (P0_4)
- net COM_M0: now also U903.12 (P0_6); no longer U903.11 (P0_5)
- net COM_M1: now also U903.13 (P0_7); no longer U903.12 (P0_6)
- net COM_P_EN: now also U903.11 (P0_5); no longer U903.15 (P1_5)
- net GND: now also SW901.2 (B)
- net MCU_CAM_EN: no longer U903.14 (P1_4)
- net VCC: now also D901.2 (A), D902.2 (A), D903.2 (A), R903.1
- net SW_SOFT: now reaches U901.31 (GPIO38/FSPIWP/SUBSPIWP)
- net SW_SOFT: now also R903.2, SW901.1 (A)
- net MC1: now reaches U901.34 (MTDI/GPIO41/CLK_OUT1)
- net MC2: now reaches U901.35 (MTMS/GPIO42)
- net at U903.1 (P1_0): now also R914.2
- net M3_P_EN: now reaches U903.17 (P1_7)
- net at U903.2 (P1_1): now also R915.2
- net at U903.3 (P1_2): now also R916.2
- net M1PG: now reaches U903.6 (P0_1)
- net M2PG: now reaches U903.7 (P0_2)
- net M3PG: now reaches U903.8 (P0_3)
- net Motor_P_EN renamed M1-2_P_EN
- new net: D902.1 (K), R915.1
- new net: D901.1 (K), R914.1
- new net: D903.1 (K), R916.1
- new net M1-2_EN: U903.15 (P1_5)
- no-connect marks 33 -> 23
Other:
- moved on the sheet: C906, U903

Commit message: Update: いろいろした
GPS変えた
USB追加した
気圧センサ変えた
FPGA変えた
MDにキャパシタ追加した
Parts:
- U903: LCSC Part (none) -> C148077
Changed lines of the file:
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@@
+			)
+		)
+		(property "LCSC Part" "C148077"
+			(at 101.6 152.4 0)
+			(hide yes)
+			(show_name no)
+			(do_not_autoplace no)
+			(effects
+				(font
+					(size 1.27 1.27)
+				)
 			)
 		)

Commit message: Update: 完成した
Parts:
- added C905: 1uF, Capacitor_SMD:C_0402_1005Metric, symbol Device:C_Small
- added C908, C909: 100nF, Capacitor_SMD:C_0402_1005Metric, symbol Device:C_Small
- added R918, R923: 200k, Resistor_SMD:R_0402_1005Metric, symbol Device:R_Small
- added R919: 150k, Resistor_SMD:R_0402_1005Metric, symbol Device:R
- added R920, R921: 4.7k, Resistor_SMD:R_0402_1005Metric, symbol Device:R
- added R924, R925: 10k, Resistor_SMD:R_0402_1005Metric, symbol Device:R
- added U904, U905: PCA9306DQER, Package_SON:X2SON-8_1.4x1mm_P0.35mm, symbol Interface:PCA9306D
- SW901: 秋月 Part (none) -> 115367
- renumbered C905 to C906, C906 to C907
Connections:
- net CAM_PIN_D0: no longer U902.4 (GPIO4/TOUCH4/ADC1_CH3)
- net CAM_PIN_D1: no longer U902.5 (GPIO5/TOUCH5/ADC1_CH4)
- net CAM_PIN_D2: no longer U902.6 (GPIO6/TOUCH6/ADC1_CH5)
- net CAM_PIN_D3: no longer U902.7 (GPIO7/TOUCH7/ADC1_CH6)
- net CAM_PIN_D4: no longer U902.8 (GPIO15/U0RTS/ADC2_CH4/XTAL_32K_P)
- net CAM_PIN_D5: no longer U902.9 (GPIO16/U0CTS/ADC2_CH5/XTAL_32K_N)
- net CAM_PIN_D6: no longer U902.10 (GPIO17/U1TXD/ADC2_CH6)
- net CAM_PIN_D7: no longer U902.11 (GPIO18/U1RXD/ADC2_CH7/CLK_OUT3)
- net CAM_PIN_HREF: no longer U902.17 (GPIO9/TOUCH9/ADC1_CH8/FSPIHD/SUBSPIHD)
- net CAM_PIN_PCLK: no longer U902.12 (GPIO8/TOUCH8/ADC1_CH7/SUBSPICS1)
- net CAM_PIN_PWDN: now also R924.2, U905.3 (SCL1); no longer U902.23 (GPIO21)
- net CAM_PIN_RESET: now also R925.2, U905.4 (SDA1); no longer U902.31 (GPIO38/FSPIWP/SUBSPIWP)
- net CAM_PIN_SIOC: now also U904.3 (SCL1); no longer U902.25 (GPIO48/SPICLK_N/SUBSPICLK_N_DIFF)
- net CAM_PIN_SIOD: now also U904.4 (SDA1); no longer U902.24 (GPIO47/SPICLK_P/SUBSPICLK_P_DIFF)
- net CAM_PIN_VSYNC: no longer U902.22 (GPIO14/TOUCH14/ADC2_CH3/FSPIWP/FSPIDQS/SUBSPIWP)
- net GND: now also C905.2, C908.2, C909.2, R919.2, U904.1 (GND), U905.1 (GND); no longer R901.2
- net MCU_CAM_EN: no longer U902.3 (EN)
- net VCC: now also R920.1, R921.1
- new net: C905.1, R901.2, U902.3 (EN)
- new net: C908.1, R918.2, U904.7 (VREF2), U904.8 (EN)
- new net: C909.1, R923.2, U905.7 (VREF2), U905.8 (EN)
- new net 1.8V: R919.1, R924.1, R925.1, U904.2 (VREF1), U905.2 (VREF1)
- new net CP_CAM_PIN_D0: U902.4 (GPIO4/TOUCH4/ADC1_CH3)
- new net CP_CAM_PIN_D1: U902.5 (GPIO5/TOUCH5/ADC1_CH4)
- new net CP_CAM_PIN_D2: U902.6 (GPIO6/TOUCH6/ADC1_CH5)
- new net CP_CAM_PIN_D3: U902.7 (GPIO7/TOUCH7/ADC1_CH6)
- new net CP_CAM_PIN_D4: U902.8 (GPIO15/U0RTS/ADC2_CH4/XTAL_32K_P)
- new net CP_CAM_PIN_D5: U902.9 (GPIO16/U0CTS/ADC2_CH5/XTAL_32K_N)
- new net CP_CAM_PIN_D6: U902.10 (GPIO17/U1TXD/ADC2_CH6)
- new net CP_CAM_PIN_D7: U902.11 (GPIO18/U1RXD/ADC2_CH7/CLK_OUT3)
- new net CP_CAM_PIN_HREF: U902.17 (GPIO9/TOUCH9/ADC1_CH8/FSPIHD/SUBSPIHD)
- new net CP_CAM_PIN_PCLK: U902.12 (GPIO8/TOUCH8/ADC1_CH7/SUBSPICS1)
- new net CP_CAM_PIN_PWDN: U902.23 (GPIO21), U905.6 (SCL2)
- new net CP_CAM_PIN_RESET: U902.31 (GPIO38/FSPIWP/SUBSPIWP), U905.5 (SDA2)
- new net CP_CAM_PIN_SIOC: R920.2, U902.25 (GPIO48/SPICLK_N/SUBSPICLK_N_DIFF), U904.6 (SCL2)
- new net CP_CAM_PIN_SIOD: R921.2, U902.24 (GPIO47/SPICLK_P/SUBSPICLK_P_DIFF), U904.5 (SDA2)
- new net CP_CAM_PIN_VSYNC: U902.22 (GPIO14/TOUCH14/ADC2_CH3/FSPIWP/FSPIDQS/SUBSPIWP)
- new net LS_EN: R918.1, R923.1
Other:
- sheet FPGA ports: added 1.8V, CP_CAM_PIN_D0, CP_CAM_PIN_D1, CP_CAM_PIN_D2, CP_CAM_PIN_D3, CP_CAM_PIN_D4, CP_CAM_PIN_D5, CP_CAM_PIN_D6, CP_CAM_PIN_D7, CP_CAM_PIN_HREF, CP_CAM_PIN_PCLK, CP_CAM_PIN_PWDN, CP_CAM_PIN_RESET, CP_CAM_PIN_VSYNC, LS_EN; removed none
- moved on the sheet: C907, D901, D902, D903, R903, R904, R905, R906, R907, R908, R909, R910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
