File: cansat2026/USB.kicad_sch (KiCad schematic)
At the start: 18 parts, among them J1101 USB_C_Receptacle_USB2.0_14P, J1102 USB_C_Receptacle_USB2.0_14P, Q1101 2N7002, Q1102 2N7002, Q1103 2N7002, Q1104 2N7002, U1101 USBLC6-2SC6, U1102 CH340K, U1103 USBLC6-2SC6, U1104 CH340K

Commit message: Update: 完成した
Parts:
- J1101, J1102: LCSC Part (none) -> C36936538
- U1101, U1103: LCSC Part (none) -> C5180249
- U1102, U1104: 秋月 Part (none) -> 116306
Changed lines of the file:
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@@
+			)
+		)
+		(property "LCSC Part" "C36936538"
+			(at 76.2 125.73 0)
+			(hide yes)
+			(show_name no)
+			(do_not_autoplace no)
+			(effects
+				(font
+					(size 1.27 1.27)
+				)
 			)
 		)
@@
 			)
 		)
+		(property "秋月 Part" "116306"
+			(at 152.4 125.73 0)
+			(hide yes)
+			(show_name no)
+			(do_not_autoplace no)
+			(effects
+				(font
+					(size 1.27 1.27)
+				)
+			)
+		)
 		(pin "8"
 		)
@@
 			)
 		)
+		(property "LCSC Part" "C36936538"
+			(at 76.2 76.2 0)
+			(hide yes)
+			(show_name no)
+			(do_not_autoplace no)
+			(effects
+				(font
+					(size 1.27 1.27)
+				)
+			)
+		)
 		(pin "B5"
 		)
@@
 			)
 		)
+		(property "秋月 Part" "116306"
+			(at 152.4 76.2 0)
+			(hide yes)
+			(show_name no)
+			(do_not_autoplace no)
+			(effects
+				(font
+					(size 1.27 1.27)
+				)
+			)
+		)
 		(pin "8"
 		)
@@
 			)
 		)
+		(property "LCSC Part" "C5180249"
+			(at 114.3 76.2 0)
+			(hide yes)
+			(show_name no)
+			(do_not_autoplace no)
+			(effects
+				(font
+					(size 1.27 1.27)
+				)
+			)
+		)
 		(pin "3"
 		)
@@
 			(at 114.3 125.73 0)
 			(hide yes)
+			(show_name no)
+			(do_not_autoplace no)
+			(effects
+				(font
+					(size 1.27 1.27)
+				)
+			)
+		)
+		(property "LCSC Part" "C5180249"
+			(at 114.3 125.73 0)
+			(hide yes)
