File: cansat2026/USB.kicad_sch (KiCad schematic)
At the start: 18 parts, among them J1101 USB_C_Receptacle_USB2.0_14P, J1102 USB_C_Receptacle_USB2.0_14P, Q1101 2N7002, Q1102 2N7002, Q1103 2N7002, Q1104 2N7002, U1101 USBLC6-2SC6, U1102 CH340K, U1103 USBLC6-2SC6, U1104 CH340K

Commit message: ARLISSに作り直した
Parts:
- removed C1103, C1104: 100nF, Capacitor_SMD:C_0402_1005Metric, symbol Device:C_Small
- removed J1102: USB_C_Receptacle_USB2.0_14P, Connector_USB:USB_C_Receptacle_GCT_USB4105-xx-A_16P_TopMnt_Horizontal, symbol Connector:USB_C_Receptacle_USB2.0_14P
- removed Q1103, Q1104: 2N7002, Package_TO_SOT_SMD:SOT-23, symbol Transistor_FET:2N7002
- removed R1103, R1104: 5.1k, Resistor_SMD:R_0402_1005Metric, symbol Device:R_Small
- removed U1103: USBLC6-2SC6, Package_TO_SOT_SMD:SOT-23-6, symbol Power_Protection:USBLC6-2SC6
- removed U1104: CH340K, Package_SO:SSOP-10-1EP_3.9x4.9mm_P1mm_EP2.1x3.3mm, symbol Interface_USB:CH340K
Connections:
- no-connect marks 2 -> 1
