File: cansat2026/FPGA.kicad_sch (KiCad schematic)
At the start: 25 parts, among them U1001 ICE40UP5K-SG48ITR

Commit message: ARLISSに作り直した
Parts:
- D1001, D1002, D1003: LCSC Part C2286 -> (none)
Connections:
- net 3.3V: no longer C1011.1, C1012.1, U1001.1 (VCCIO_2)
- net CAM_PIN_PWDN: now reaches U1001.44 (IOB_3b_G6)
- net CAM_PIN_RESET: now reaches U1001.45 (IOB_5b)
- net CAM_PIN_SIOD: now reaches U1001.47 (IOB_2a)
- net at C1007.1, C1008.1, JP1001.2 (C)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: now also C1011.1, C1012.1, U1001.1 (VCCIO_2)
- net CP_CAM_PIN_D0: no longer names the net of U1001.6 (IOB_13b)
- net CP_CAM_PIN_D1: no longer names the net of U1001.9 (IOB_16a)
- net CP_CAM_PIN_D2: no longer names the net of U1001.10 (IOB_18a)
- net CP_CAM_PIN_D3: no longer names the net of U1001.11 (IOB_20a)
- net CP_CAM_PIN_D4: no longer names the net of U1001.12 (IOB_22a)
- net CP_CAM_PIN_D5: no longer names the net of U1001.21 (IOB_23b)
- net CP_CAM_PIN_D6: no longer names the net of U1001.13 (IOB_24a)
- net CP_CAM_PIN_D7: no longer names the net of U1001.18 (IOB_31b)
- net CP_CAM_PIN_HREF: no longer names the net of U1001.19 (IOB_29b)
- net CP_CAM_PIN_PCLK: no longer names the net of U1001.20 (IOB_25b_G3)
- net CP_CAM_PIN_PWDN: no longer names the net of U1001.4 (IOB_8a)
- net CP_CAM_PIN_RESET: no longer names the net of U1001.3 (IOB_9b)
- net CP_CAM_PIN_VSYNC: no longer names the net of U1001.2 (IOB_6a)
- net LS_EN renamed CAM_PIN_SIOC
- no-connect marks 6 -> 16
Changed lines of the file:
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@@
 	)
 	(junction
+		(at 58.42 50.8)
+		(diameter 0)
+		(color 0 0 0 0)
+	)
+	(junction
 		(at 186.69 55.88)
 		(diameter 0)
@@
 	)
 	(junction
+		(at 148.59 50.8)
+		(diameter 0)
+		(color 0 0 0 0)
+	)
+	(junction
 		(at 15.24 104.14)
 		(diameter 0)
@@
 	)
 	(no_connect
-		(at 158.75 83.82)
+		(at 158.75 88.9)
 	)
 	(no_connect
-		(at 48.26 101.6)
+		(at 107.95 101.6)
+	)
+	(no_connect
+		(at 107.95 88.9)
+	)
+	(no_connect
+		(at 107.95 86.36)
 	)
 	(no_connect
-		(at 158.75 78.74)
+		(at 107.95 83.82)
 	)
 	(no_connect
@@
 	)
 	(no_connect
-		(at 158.75 76.2)
+		(at 48.26 101.6)
+	)
+	(no_connect
+		(at 107.95 96.52)
+	)
+	(no_connect
+		(at 158.75 86.36)
+	)
+	(no_connect
+		(at 107.95 78.74)
+	)
+	(no_connect
+		(at 107.95 91.44)
+	)
+	(no_connect
+		(at 158.75 91.44)
+	)
+	(no_connect
+		(at 107.95 99.06)
+	)
+	(no_connect
+		(at 107.95 81.28)
+	)
+	(no_connect
+		(at 107.95 93.98)
 	)
 	(wire
@@
 	(wire
 		(pts
+			(xy 58.42 45.72) (xy 148.59 45.72)
+		)
+		(stroke
+			(width 0)
+			(type default)
+		)
+	)
+	(wire
+		(pts
 			(xy 97.79 55.88) (xy 109.22 55.88)
 		)
@@
 	(wire
 		(pts
+			(xy 148.59 45.72) (xy 148.59 50.8)
+		)
+		(stroke
+			(width 0)
+			(type default)
+		)
+	)
+	(wire
+		(pts
 			(xy 97.79 58.42) (xy 97.79 55.88)
 		)
@@
 	(wire
 		(pts
+			(xy 58.42 50.8) (xy 58.42 45.72)
+		)
+		(stroke
+			(width 0)
+			(type default)
+		)
+	)
+	(wire
+		(pts
 			(xy 196.85 38.1) (xy 208.28 38.1)
 		)
@@
 	)
 	(label "3.3V"
-		(at 148.59 50.8 180)
-		(effects
-			(font
-				(size 1.27 1.27)
-			)
-			(justify right bottom)
-		)
-	)
-	(label "3.3V"
 		(at 186.69 50.8 180)
 		(effects
@@
 		)
 	)
-	(hierarchical_label "CP_CAM_PIN_D6"
-		(shape output)
-		(at 107.95 93.98 180)
-		(effects
-			(font
-				(size 1.27 1.27)
-			)
-			(justify right)
-		)
-	)
 	(hierarchical_label "SPI_SO"
 		(shape output)
@@
 		)
 	)
-	(hierarchical_label "CP_CAM_PIN_RESET"
-		(shape output)
-		(at 158.75 91.44 180)
-		(effects
-			(font
-				(size 1.27 1.27)
-			)
-			(justify right)
-		)
-	)
-	(hierarchical_label "CP_CAM_PIN_D1"
-		(shape output)
-		(at 107.95 81.28 180)
-		(effects
-			(font
-				(size 1.27 1.27)
-			)
-			(justify right)
-		)
-	)
 	(hierarchical_label "CAM_PIN_D6"
 		(shape input)
@@
 		)
 	)
-	(hierarchical_label "CP_CAM_PIN_PCLK"
+	(hierarchical_label "CAM_PIN_SIOC"
 		(shape output)
-		(at 107.95 96.52 180)
+		(at 158.75 73.66 180)
 		(effects
 			(font
@@
 		)
 	)
-	(hierarchical_label "CAM_PIN_D3"
-		(shape input)
-		(at 48.26 78.74 180)
+	(hierarchical_label "CAM_PIN_PWDN"
+		(shape output)
+		(at 158.75 78.74 180)
 		(effects
 			(font
@@
 		)
 	)
-	(hierarchical_label "CP_CAM_PIN_PWDN"
-		(shape output)
-		(at 158.75 88.9 180)
+	(hierarchical_label "CAM_PIN_D3"
+		(shape input)
+		(at 48.26 78.74 180)
 		(effects
 			(font
@@
 		)
 	)
-	(hierarchical_label "LS_EN"
-		(shape output)
-		(at 158.75 73.66 180)
+	(hierarchical_label "CAM_PIN_SIOD"
+		(shape bidirectional)
+		(at 158.75 76.2 180)
 		(effects
 			(font
@@
 		)
 	)
-	(hierarchical_label "CP_CAM_PIN_D4"
-		(shape output)
-		(at 107.95 88.9 180)
-		(effects
-			(font
-				(size 1.27 1.27)
-			)
-			(justify right)
-		)
-	)
-	(hierarchical_label "CP_CAM_PIN_D0"
-		(shape output)
-		(at 107.95 78.74 180)
-		(effects
-			(font
-				(size 1.27 1.27)
-			)
-			(justify right)
-		)
-	)
-	(hierarchical_label "CP_CAM_PIN_D2"
-		(shape output)
-		(at 107.95 83.82 180)
-		(effects
-			(font
-				(size 1.27 1.27)
-			)
-			(justify right)
-		)
-	)
 	(hierarchical_label "CAM_PIN_HREF"
 		(shape input)
@@
 		)
 	)
-	(hierarchical_label "CP_CAM_PIN_VSYNC"
-		(shape output)
-		(at 158.75 86.36 180)
-		(effects
-			(font
-				(size 1.27 1.27)
-			)
-			(justify right)
-		)
-	)
 	(hierarchical_label "GND"
 		(shape input)
@@
 		)
 	)
-	(hierarchical_label "CP_CAM_PIN_D7"
+	(hierarchical_label "CAM_PIN_RESET"
 		(shape output)
-		(at 107.95 101.6 180)
+		(at 158.75 83.82 180)
 		(effects
 			(font
@@
 		)
 	)
-	(hierarchical_label "CP_CAM_PIN_D5"
-		(shape output)
-		(at 107.95 91.44 180)
-		(effects
-			(font
-				(size 1.27 1.27)
-			)
-			(justify right)
-		)
-	)
 	(hierarchical_label "CAM_PIN_PCLK"
 		(shape input)
@@
 		)
 	)
-	(hierarchical_label "CP_CAM_PIN_D3"
-		(shape output)
-		(at 107.95 86.36 180)
-		(effects
-			(font
-				(size 1.27 1.27)
-			)
-			(justify right)
-		)
-	)
-	(hierarchical_label "CP_CAM_PIN_HREF"
-		(shape output)
-		(at 107.95 99.06 180)
-		(effects
-			(font
-				(size 1.27 1.27)
-			)
-			(justify right)
-		)
-	)
 	(hierarchical_label "CAM_PIN_D7"
 		(shape input)
@@
 		(in_pos_files yes)
 		(dnp no)
-		(fields_autoplaced yes)
 		(property "Reference" "C1004"
 			(at 187.96 39.3762 0)
@@
 			)
 		)
-		(property "LCSC Part" "C2286"
+		(property "LCSC Part" ""
 			(at 15.24 106.68 0)
 			(hide yes)
@@
 			)
 		)
-		(property "LCSC Part" "C2286"
+		(property "LCSC Part" ""
 			(at 25.4 106.68 0)
 			(hide yes)
@@
 			)
 		)
-		(property "LCSC Part" "C2286"
+		(property "LCSC Part" ""
 			(at 35.56 106.68 0)
 			(hide yes)
