File: cansat2026/GPS.kicad_sch (KiCad schematic)
At the start: 11 parts, among them J801 Conn_Coaxial, U801 MAX-M10S

Commit message: ARLISSに作り直した
Parts:
- L801: LCSC Part (none) -> C148128
Connections:
- net SCL: no longer names the net of U801.17 (SCL)
- net SDA: no longer names the net of U801.16 (SDA)
- no-connect marks 5 -> 7
Changed lines of the file:
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@@
+	)
+	(no_connect
+		(at 124.46 104.14)
 	)
 	(no_connect
@@
 	)
 	(no_connect
+		(at 124.46 106.68)
+	)
+	(no_connect
 		(at 124.46 111.76)
 	)
@@
 	(wire
 		(pts
-			(xy 115.57 104.14) (xy 124.46 104.14)
-		)
-		(stroke
-			(width 0)
-			(type default)
-		)
-	)
-	(wire
-		(pts
 			(xy 177.8 81.28) (xy 190.5 81.28)
-		)
-		(stroke
-			(width 0)
-			(type default)
-		)
-	)
-	(wire
-		(pts
-			(xy 115.57 106.68) (xy 124.46 106.68)
 		)
 		(stroke
@@
 			)
 			(justify left bottom)
-		)
-	)
-	(hierarchical_label "SCL"
-		(shape input)
-		(at 115.57 106.68 180)
-		(effects
-			(font
-				(size 1.27 1.27)
-			)
-			(justify right)
 		)
 	)
@@
 		(shape input)
 		(at 111.76 83.82 180)
-		(effects
-			(font
-				(size 1.27 1.27)
-			)
-			(justify right)
-		)
-	)
-	(hierarchical_label "SDA"
-		(shape bidirectional)
-		(at 115.57 104.14 180)
 		(effects
 			(font
@@
 			)
 		)
-		(property "LCSC Part" ""
+		(property "LCSC Part" "C148128"
 			(at 194.31 81.28 90)
 			(hide yes)
