File: cansat2026/MD.kicad_sch (KiCad schematic)
At the start: 18 parts, among them J401 M1, J402 M2, J403 M3, U401 TC78H653FTG, U402 TC78H653FTG, U403 AM8068

Commit message: ARLISSに作り直した
Parts:
- removed C412: 10uF, Capacitor_SMD:C_0603_1608Metric, symbol Device:C_Small
- added C412, C413, C414, C415, C416, C417: 100uF, Project:MURATA_ECAS_D6, symbol Device:C_Polarized_Small
- added C418: 22uF, Capacitor_SMD:C_0805_2012Metric, symbol Device:C_Small
- C410, C411: footprint Capacitor_THT:CP_Radial_D6.3mm_P2.50mm -> Project:MURATA_ECAS_D6; 秋月 Part 108290 -> 117422
- U401, U402: LCSC Part C37313337 -> C2150463
Connections:
- net GND: now also C412.2, C413.2, C414.2, C415.2, C416.2, C417.2, C418.2
- net M1PWR: now also C411.1, C412.1, C413.1
- net M2PWR: now also C414.1, C415.1, C416.1, C417.1; no longer C411.1
- net M3PWR: now also C418.1
