File: cansat2026/Power.kicad_sch (KiCad schematic)
At the start: 85 parts, among them J201 FlightPin, SW201 SW_SPST, U201 TPS70912DRVR, U202 TCR2LN18, U203 TPS561201DDC, U204 74HC08, U205 INA226, U206 TPS562242, U207 XC6206P332MR, U208 TPS62180, U209 TPS62180, U210 TPS63070

Commit message: ARLISSに作り直した
Parts:
- D201: LCSC Part C2286 -> (none)
- L201: footprint Inductor_SMD:L_Wuerth_PMCI-252012 -> Inductor_SMD:L_1008_2520Metric_Pad1.43x2.20mm_HandSolder
- L202: footprint Inductor_SMD:L_Taiyo-Yuden_NR-50xx -> Inductor_SMD:L_Taiyo-Yuden_NR-50xx_HandSoldering
- L203, L204, L205, L206: footprint Inductor_SMD:L_Wuerth_PMCI-252010 -> Project:L_Taiyo-Yuden_LSEU-4040; DigiKey Part CIGT252010EH1R0MNE -> (none); Mouser Part 810-VLS6045EX-3R3N -> 963-LSEUB4040WKT1R0M
- L207: footprint Inductor_SMD:L_Wuerth_PMCI-201610 -> Project:L_Wuerth_PMCI-201610
- R204, R209: LCSC Part C25007 -> C25077
- R216, R219: LCSC Part C25774 -> C25755
- RV201, RV202: LCSC Part (none) -> C5361820
Changed lines of the file:
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@@
 			)
 		)
-		(property "Footprint" "Inductor_SMD:L_Wuerth_PMCI-252010"
+		(property "Footprint" "Project:L_Taiyo-Yuden_LSEU-4040"
 			(at 156.21 134.62 0)
 			(hide yes)
@@
 			)
 		)
-		(property "Mouser Part" "810-VLS6045EX-3R3N"
+		(property "Mouser Part" "963-LSEUB4040WKT1R0M "
 			(at 156.21 134.62 90)
 			(hide yes)
@@
 			)
 		)
-		(property "DigiKey Part" "CIGT252010EH1R0MNE"
+		(property "DigiKey Part" ""
 			(at 156.21 134.62 90)
 			(hide yes)
@@
 			)
 		)
-		(property "LCSC Part" "C25774"
+		(property "LCSC Part" "C25755"
 			(at 179.07 146.05 0)
 			(hide yes)
@@
 			)
 		)
-		(property "LCSC Part" "C2286"
+		(property "LCSC Part" ""
 			(at 214.63 72.39 90)
 			(hide yes)
@@
 			)
 		)
-		(property "LCSC Part" "C25007"
+		(property "LCSC Part" "C25077"
 			(at 27.94 71.12 90)
 			(hide yes)
@@
 			)
 		)
-		(property "Footprint" "Inductor_SMD:L_Wuerth_PMCI-252010"
+		(property "Footprint" "Project:L_Taiyo-Yuden_LSEU-4040"
 			(at 156.21 127 0)
 			(hide yes)
@@
 			)
 		)
-		(property "Mouser Part" "810-VLS6045EX-3R3N"
+		(property "Mouser Part" "963-LSEUB4040WKT1R0M "
 			(at 156.21 127 90)
 			(hide yes)
@@
 			)
 		)
-		(property "DigiKey Part" "CIGT252010EH1R0MNE"
+		(property "DigiKey Part" ""
 			(at 156.21 127 90)
 			(hide yes)
@@
 			)
 		)
-		(property "Footprint" "Inductor_SMD:L_Wuerth_PMCI-252012"
+		(property "Footprint" "Inductor_SMD:L_1008_2520Metric_Pad1.43x2.20mm_HandSolder"
 			(at 156.21 38.1 0)
 			(hide yes)
@@
 			)
 		)
+		(property "LCSC Part" "C5361820"
+			(at 181.61 104.14 0)
+			(hide yes)
+			(show_name no)
+			(do_not_autoplace no)
+			(effects
+				(font
+					(size 1.27 1.27)
+				)
+			)
+		)
 		(pin "3"
 		)
@@
 			)
 		)
-		(property "Footprint" "Inductor_SMD:L_Taiyo-Yuden_NR-50xx"
+		(property "Footprint" "Inductor_SMD:L_Taiyo-Yuden_NR-50xx_HandSoldering"
 			(at 156.21 68.58 0)
 			(hide yes)
@@
 			)
 		)
-		(property "Footprint" "Inductor_SMD:L_Wuerth_PMCI-201610"
+		(property "Footprint" "Project:L_Wuerth_PMCI-201610"
 			(at 124.46 177.8 0)
 			(hide yes)
@@
 			)
 		)
-		(property "Footprint" "Inductor_SMD:L_Wuerth_PMCI-252010"
+		(property "Footprint" "Project:L_Taiyo-Yuden_LSEU-4040"
 			(at 156.21 104.14 0)
 			(hide yes)
@@
 			)
 		)
-		(property "Mouser Part" "810-VLS6045EX-3R3N"
+		(property "Mouser Part" "963-LSEUB4040WKT1R0M "
 			(at 156.21 104.14 90)
 			(hide yes)
@@
 			)
 		)
-		(property "DigiKey Part" "CIGT252010EH1R0MNE"
+		(property "DigiKey Part" ""
 			(at 156.21 104.14 90)
 			(hide yes)
@@
 			)
 		)
+		(property "LCSC Part" "C5361820"
+			(at 181.61 134.62 0)
+			(hide yes)
+			(show_name no)
+			(do_not_autoplace no)
+			(effects
+				(font
+					(size 1.27 1.27)
+				)
+			)
+		)
 		(pin "3"
 		)
@@
 			)
 		)
-		(property "Footprint" "Inductor_SMD:L_Wuerth_PMCI-252010"
+		(property "Footprint" "Project:L_Taiyo-Yuden_LSEU-4040"
 			(at 156.21 96.52 0)
 			(hide yes)
@@
 			)
 		)
-		(property "Mouser Part" "810-VLS6045EX-3R3N"
+		(property "Mouser Part" "963-LSEUB4040WKT1R0M "
 			(at 156.21 96.52 90)
 			(hide yes)
@@
 			)
 		)
-		(property "DigiKey Part" "CIGT252010EH1R0MNE"
+		(property "DigiKey Part" ""
 			(at 156.21 96.52 90)
 			(hide yes)
@@
 			)
 		)
-		(property "LCSC Part" "C25774"
+		(property "LCSC Part" "C25755"
 			(at 179.07 115.57 0)
 			(hide yes)
@@
 			)
 		)
-		(property "LCSC Part" "C25007"
+		(property "LCSC Part" "C25077"
 			(at 27.94 78.74 90)
 			(hide yes)
