File: cansat2026/cansat2026.kicad_sch (KiCad schematic)
At the start: 12 parts, among them J101 MCU_UART_Conn, J102 CAM_Conn, J103 MCU_CAM_UART_Conn, J104 I2C_Conn, J105 MCU_Power, J106 MCU_Power, J107 Micro_SD_Card_Det_Hirose_DM3AT, U101 E220-900T22S(JP)

Commit message: ARLISSに作り直した
Parts:
- removed J103: MCU_CAM_UART_Conn, Connector_PinSocket_2.54mm:PinSocket_1x05_P2.54mm_Vertical, symbol Connector:Conn_01x05_Socket
- renumbered J104 to J103, J105 to J104, J106 to J105, J107 to J106
Other:
- sheet GPS ports: added none; removed SCL, SDA
- sheet MCU ports: added none; removed MCU_CAM_EN, MCU_CAM_GPIO0, MCU_CAM_U0RXD, MCU_CAM_U0TXD
